File: schema's/Shield_behuizing.sch (EAGLE design)
At the start: 5 parts, among them U1 CCS811

Commit message: pcb gemaakt
Parts:
- added BATT1, BATT2, BATT3, BATT4, BATT5, BATT6: AAA, adafruit:AAA
- added U$5: GPS-RECEIVER-NEO6M, diy-modules:GPS-RECEIVER-NEO6M
- added X1, X2: 87758-0216, con-molex:87758-0216
Connections:
- new net N$10: BATT2.+, BATT3.-
- new net N$11: BATT3.+, BATT4.-
- new net N$12: BATT4.+, BATT5.-
- new net N$13: BATT5.+, BATT6.-
- new net N$14: U$2.3V, U$4.VCC, U$5.VCC, U1.VDD
- new net N$15: U$2.D4, U$5.TXD
- new net N$16: BATT1.-, X1-1.S, X2-1.S
- new net N$17: BATT6.+, X1-2.S, X2-2.S
- new net N$18: U$2.D3, U$5.RXD
- new net N$4: BATT1.+, BATT2.-
- net N$5: now also U$4.ADDR, U$5.GND, U1.ADDR
- net N$9: no longer U$4.VCC, U1.VDD
