File: schema's/GIP-client.sch (EAGLE design)
At the start: 14 parts, among them U1 CCS811, X1 87758-0216, X2 87758-0216

Commit message: pcb gemaakt
Parts:
- removed BATT1, BATT2, BATT3, BATT4, BATT5, BATT6: AAA, adafruit:AAA
- removed U$1: GSM-MODEM-SIM900A, diy-modules:GSM-MODEM-SIM900A
- removed U1: CCS811, CCS811_Breakout_Temp:CCS811
- removed X1: 87758-0216, con-molex:87758-0216
- added SV1: (no value), con-lstb:MA06-1
- X2: value 87758-0216 -> (none); device con-molex:87758-0216 -> con-phoenix-254:MPT3
Connections:
- removed net N$10: BATT2.+, BATT3.-
- removed net N$11: BATT3.+, BATT4.-
- removed net N$12: BATT4.+, BATT5.-
- removed net N$13: BATT5.+, BATT6.-
- removed net N$16: BATT1.-, X1-1.S, X2-1.S
- removed net N$17: BATT6.+, X1-2.S, X2-2.S
- removed net N$4: BATT1.+, BATT2.-
- net N$1: now also X2-1.1; no longer U$1.GND.1
- net N$14: now also SV1.5; no longer U1.VDD
- net N$2: now also X2-2.1; no longer U$1.SIMR
- net N$3: now also X2-3.1; no longer U$1.SIMT
- net N$5: now also SV1.1, SV1.2, SV1.6; no longer U1.!WAKE!, U1.ADDR, U1.GND
- net N$7: now also SV1.4; no longer U1.SDA
- net N$8: now also SV1.3; no longer U1.SCL

Commit message: pcb
Connections:
- net N$14: no longer U$4.VCC
- net N$9: now also U$4.VCC
Changed lines of the file:
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@@
 <wire x1="-20.32" y1="43.18" x2="-20.32" y2="40.64" width="0.1524" layer="91"/>
 <wire x1="-20.32" y1="40.64" x2="-5.08" y2="40.64" width="0.1524" layer="91"/>
+<pinref part="U$4" gate="G$1" pin="VCC"/>
+<wire x1="-27.94" y1="27.94" x2="-5.08" y2="27.94" width="0.1524" layer="91"/>
+<wire x1="-5.08" y1="27.94" x2="-5.08" y2="40.64" width="0.1524" layer="91"/>
+<junction x="-5.08" y="40.64"/>
 </segment>
 </net>
 <net name="N$14" class="0">
 <segment>
-<wire x1="-15.24" y1="5.08" x2="-15.24" y2="27.94" width="0.1524" layer="91"/>
 <pinref part="U$2" gate="G$1" pin="3V"/>
-<wire x1="-15.24" y1="27.94" x2="-15.24" y2="50.8" width="0.1524" layer="91"/>
+<wire x1="-15.24" y1="5.08" x2="-15.24" y2="50.8" width="0.1524" layer="91"/>
 <wire x1="-15.24" y1="50.8" x2="5.08" y2="50.8" width="0.1524" layer="91"/>
-<pinref part="U$4" gate="G$1" pin="VCC"/>
-<wire x1="-27.94" y1="27.94" x2="-15.24" y2="27.94" width="0.1524" layer="91"/>
-<junction x="-15.24" y="27.94"/>
 <pinref part="U$5" gate="G$1" pin="VCC"/>
 <wire x1="-15.24" y1="5.08" x2="93.98" y2="5.08" width="0.1524" layer="91"/>
@@
 <wire x1="-50.8" y1="0" x2="-15.24" y2="0" width="0.1524" layer="91"/>
 <wire x1="-15.24" y1="0" x2="-15.24" y2="5.08" width="0.1524" layer="91"/>
+<junction x="-15.24" y="5.08"/>
 </segment>
 </net>
