File: schema's/GIP-client.brd (EAGLE design)
At the start: 100 x 80 mm, 8 parts, among them U1 CCS811, X1 87758-0216, X2 87758-0216

Commit message: pcb gemaakt
Parts:
- removed U$1: GSM-MODEM-SIM900A, diy-modules:GSM-MODEM-SIM900A
- removed U1: CCS811, CCS811_Breakout_Temp:LGA10
- removed X1: 87758-0216, con-molex:87758-0216
- added SV1: (no value), con-lstb:MA06-1
- X2: value 87758-0216 -> (none); device con-molex:87758-0216 -> con-phoenix-254:3POL254
- moved X2 132.0 mm to (43.2, 64.8)
- moved U$2 104.6 mm to (14.0, 17.8)
- moved U$5 57.4 mm to (39.4, 40.6)
- moved U$3 50.1 mm to (67.3, 25.4), turned to 0 degrees
- moved U$4 43.8 mm to (73.7, 68.6)
Connections:
- removed net GND.2: U$1.J1.7
- removed net VCC4: U$1.J1.3
- removed net VCC5: U$1.J1.1
- removed net VCCMCU: U$1.J1.4
- net N$1: now also X2.1; no longer U$1.J1.2
- net N$14: now also SV1.5; no longer U1.6
- net N$2: now also X2.2; no longer U$1.J1.5
- net N$3: now also X2.3; no longer U$1.J1.6
- net N$5: now also SV1.1, SV1.2, SV1.6; no longer U1.1, U1.7, U1.EP
- net N$7: now also SV1.4; no longer U1.9
- net N$8: now also SV1.3; no longer U1.10
Routing:
- net N$5: track 0.00 -> 102.9 mm
- net N$14: track 0.00 -> 92.4 mm
- net N$18: track 0.00 -> 55.5 mm
- net N$15: track 0.00 -> 55.5 mm
- net N$7: track 0.00 -> 46.5 mm
- net N$6: track 0.00 -> 44.9 mm
- net N$8: track 0.00 -> 44.3 mm
- net N$3: track 0.00 -> 15.6 mm
- net N$2: track 0.00 -> 14.1 mm
- net N$9: track 0.00 -> 13.5 mm
- net N$1: track 0.00 -> 3.97 mm

Commit message: pcb
Parts:
- moved SV1 16.6 mm to (66.0, 49.5)
- moved U$2 16.6 mm to (0.00, 26.7)
- moved U$3 16.6 mm to (53.3, 34.3)
- moved U$4 16.6 mm to (59.7, 77.5)
- moved U$5 16.6 mm to (25.4, 49.5)
- moved X2 16.6 mm to (29.2, 73.7)
Connections:
- net N$14: no longer U$4.1
- net N$9: now also U$4.1
Routing:
- net N$6: track 44.9 -> 104.4 mm
- net N$9: track 13.5 -> 64.2 mm
- net N$8: track 44.3 -> 72.6 mm
- net N$5: track 102.9 -> 129.3 mm
- net N$14: track 92.4 -> 100.5 mm
- net N$18: track 55.5 -> 61.9 mm
- net N$15: track 55.5 -> 60.7 mm
Other:
- board size 100 x 80 mm -> 69.5 x 53.3 mm

Commit message: Pcb afgemaakt
Other:
- board size 69.5 x 53.3 mm -> 56.8 x 53.3 mm
Changed lines of the file:
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@@
 <board>
 <plain>
-<wire x1="0" y1="26.67" x2="69.52" y2="26.67" width="0" layer="20"/>
+<wire x1="12.7" y1="26.67" x2="69.52" y2="26.67" width="0" layer="20"/>
 <wire x1="69.52" y1="26.67" x2="69.52" y2="80" width="0" layer="20"/>
-<wire x1="69.52" y1="80" x2="0" y2="80" width="0" layer="20"/>
-<wire x1="0" y1="80" x2="0" y2="26.67" width="0" layer="20"/>
+<wire x1="69.52" y1="80" x2="12.7" y2="80" width="0" layer="20"/>
+<wire x1="12.7" y1="80" x2="12.7" y2="26.67" width="0" layer="20"/>
 </plain>
 <attributes>

Commit message: gerber files voor pcb
Routing:
- net N$14: track 100.5 -> 110.4 mm
- net N$9: track 64.2 -> 68.3 mm
- net N$18: track 61.9 -> 64.3 mm
- net N$5: track 129.3 -> 131.4 mm
Changed lines of the file:
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@@
 <?xml version="1.0" encoding="utf-8"?>
 <!DOCTYPE eagle SYSTEM "eagle.dtd">
-<eagle version="7.1.0">
+<eagle version="9.0.1">
 <drawing>
 <settings>
-<setting alwaysvectorfont="no"/>
+<setting alwaysvectorfont="yes"/>
+<setting keepoldvectorfont="yes"/>
 <setting verticaltext="up"/>
 </settings>
@@
 <layer number="59" name="tCarbon" color="7" fill="1" visible="no" active="no"/>
 <layer number="60" name="bCarbon" color="7" fill="1" visible="no" active="no"/>
-<layer number="88" name="SimResults" color="9" fill="1" visible="yes" active="yes"/>
-<layer number="89" name="SimProbes" color="9" fill="1" visible="yes" active="yes"/>
+<layer number="88" name="SimResults" color="9" fill="1" visible="no" active="no"/>
+<layer number="89" name="SimProbes" color="9" fill="1" visible="no" active="no"/>
 <layer number="90" name="Modules" color="5" fill="1" visible="no" active="no"/>
 <layer number="91" name="Nets" color="2" fill="1" visible="no" active="no"/>
@@
 <param name="dpMaxLengthDifference" value="10mm"/>
 <param name="dpGapFactor" value="2.5"/>
-<param name="checkGrid" value="0"/>
 <param name="checkAngle" value="0"/>
 <param name="checkFont" value="1"/>
 <param name="checkRestrict" value="1"/>
+<param name="checkStop" value="0"/>
+<param name="checkValues" value="0"/>
 <param name="useDiameter" value="13"/>
 <param name="maxErrors" value="50"/>
@@
 <element name="U$5" library="diy-modules" package="GPS-RECEIVER-NEO6M" value="GPS-RECEIVER-NEO6M" x="25.4" y="49.53" rot="R90"/>
 <element name="SV1" library="con-lstb" package="MA06-1" value="" x="66.04" y="49.53" rot="R90">
+<attribute name="MF" value="" x="66.04" y="49.53" size="1.778" layer="27" rot="R90" display="off"/>
+<attribute name="MPN" value="" x="66.04" y="49.53" size="1.778" layer="27" rot="R90" display="off"/>
+<attribute name="OC_FARNELL" value="unknown" x="66.04" y="49.53" size="1.778" layer="27" rot="R90" display="off"/>
 <attribute name="OC_NEWARK" value="unknown" x="66.04" y="49.53" size="1.778" layer="27" rot="R90" display="off"/>
-<attribute name="MPN" value="" x="66.04" y="49.53" size="1.778" layer="27" rot="R90" display="off"/>
-<attribute name="MF" value="" x="66.04" y="49.53" size="1.778" layer="27" rot="R90" display="off"/>
-<attribute name="OC_FARNELL" value="unknown" x="66.04" y="49.53" size="1.778" layer="27" rot="R90" display="off"/>
 </element>
 <element name="X2" library="con-phoenix-254" package="3POL254" value="" x="29.21" y="73.66">
+<attribute name="MF" value="" x="29.21" y="73.66" size="1.778" layer="27" display="off"/>
+<attribute name="MPN" value="" x="29.21" y="73.66" size="1.778" layer="27" display="off"/>
+<attribute name="OC_FARNELL" value="unknown" x="29.21" y="73.66" size="1.778" layer="27" display="off"/>
 <attribute name="OC_NEWARK" value="unknown" x="29.21" y="73.66" size="1.778" layer="27" display="off"/>
-<attribute name="MPN" value="" x="29.21" y="73.66" size="1.778" layer="27" display="off"/>
-<attribute name="MF" value="" x="29.21" y="73.66" size="1.778" layer="27" display="off"/>
-<attribute name="OC_FARNELL" value="unknown" x="29.21" y="73.66" size="1.778" layer="27" display="off"/>
 </element>
 </elements>
@@
 <contactref element="SV1" pad="2"/>
 <contactref element="SV1" pad="1"/>
-<wire x1="56.261" y1="71.5518" x2="54.6608" y2="69.9516" width="0.254" layer="16"/>
-<wire x1="60.6044" y1="71.5518" x2="56.261" y2="71.5518" width="0.254" layer="16"/>
-<wire x1="62.2046" y1="69.9516" x2="60.6044" y2="71.5518" width="0.254" layer="16"/>
+<wire x1="56.261" y1="72.8218" x2="54.6608" y2="69.9516" width="0.254" layer="16"/>
+<wire x1="60.6044" y1="72.8218" x2="56.261" y2="72.8218" width="0.254" layer="16"/>
+<wire x1="62.2046" y1="69.9516" x2="60.6044" y2="72.8218" width="0.254" layer="16"/>
 <wire x1="54.6608" y1="69.9516" x2="54.61" y2="69.85" width="0.254" layer="16"/>
 <wire x1="62.2046" y1="69.9516" x2="62.23" y2="69.85" width="0.254" layer="16"/>
@@
 <wire x1="28.3718" y1="32.4612" x2="27.4574" y2="32.4612" width="0.254" layer="16"/>
 <wire x1="29.2862" y1="33.3756" x2="28.3718" y2="32.4612" width="0.254" layer="16"/>
-<wire x1="29.2862" y1="54.864" x2="29.2862" y2="33.3756" width="0.254" layer="16"/>
-<wire x1="48.26" y1="73.8378" x2="29.2862" y2="54.864" width="0.254" layer="16"/>
-<wire x1="48.26" y1="77.47" x2="48.26" y2="73.8378" width="0.254" layer="16"/>
+<wire x1="29.2862" y1="56.134" x2="29.2862" y2="33.3756" width="0.254" layer="16"/>
+<wire x1="48.26" y1="75.1078" x2="29.2862" y2="56.134" width="0.254" layer="16"/>
+<wire x1="48.26" y1="77.47" x2="48.26" y2="75.1078" width="0.254" layer="16"/>
 <wire x1="51.9176" y1="34.29" x2="52.07" y2="34.29" width="0.254" layer="16"/>
 </signal>
@@
 <wire x1="38.2016" y1="29.2608" x2="38.1" y2="29.21" width="0.254" layer="16"/>
 <wire x1="63.8048" y1="69.9516" x2="64.7192" y2="69.9516" width="0.254" layer="16"/>
-<wire x1="61.7474" y1="72.009" x2="63.8048" y2="69.9516" width="0.254" layer="16"/>
-<wire x1="55.118" y1="72.009" x2="61.7474" y2="72.009" width="0.254" layer="16"/>
-<wire x1="49.6316" y1="66.5226" x2="55.118" y2="72.009" width="0.254" layer="16"/>
+<wire x1="61.7474" y1="74.549" x2="63.8048" y2="69.9516" width="0.254" layer="16"/>
+<wire x1="55.118" y1="74.549" x2="61.7474" y2="74.549" width="0.254" layer="16"/>
+<wire x1="49.6316" y1="66.5226" x2="55.118" y2="74.549" width="0.254" layer="16"/>
 <wire x1="49.6316" y1="34.29" x2="49.6316" y2="66.5226" width="0.254" layer="16"/>
 <wire x1="64.7192" y1="69.9516" x2="64.77" y2="69.85" width="0.254" layer="16"/>
@@
 <wire x1="35.4584" y1="29.2608" x2="35.56" y2="29.21" width="0.254" layer="16"/>
 <wire x1="63.119" y1="56.2356" x2="65.8622" y2="53.4924" width="0.254" layer="16"/>
-<wire x1="63.119" y1="66.0654" x2="63.119" y2="56.2356" width="0.254" layer="16"/>
-<wire x1="65.8622" y1="68.8086" x2="63.119" y2="66.0654" width="0.254" layer="16"/>
-<wire x1="65.8622" y1="70.866" x2="65.8622" y2="68.8086" width="0.254" layer="16"/>
-<wire x1="64.262" y1="72.4662" x2="65.8622" y2="70.866" width="0.254" layer="16"/>
-<wire x1="54.8894" y1="72.4662" x2="64.262" y2="72.4662" width="0.254" layer="16"/>
-<wire x1="37.2872" y1="54.864" x2="54.8894" y2="72.4662" width="0.254" layer="16"/>
-<wire x1="37.2872" y1="33.3756" x2="37.2872" y2="54.864" width="0.254" layer="16"/>
+<wire x1="63.119" y1="63.5254" x2="63.119" y2="56.2356" width="0.254" layer="16"/>
+<wire x1="68.4022" y1="67.5386" x2="63.119" y2="63.5254" width="0.254" layer="16"/>
+<wire x1="68.4022" y1="70.866" x2="68.4022" y2="67.5386" width="0.254" layer="16"/>
+<wire x1="64.262" y1="76.2762" x2="68.4022" y2="70.866" width="0.254" layer="16"/>
+<wire x1="54.8894" y1="76.2762" x2="64.262" y2="76.2762" width="0.254" layer="16"/>
+<wire x1="37.2872" y1="58.674" x2="54.8894" y2="76.2762" width="0.254" layer="16"/>
+<wire x1="37.2872" y1="33.3756" x2="37.2872" y2="58.674" width="0.254" layer="16"/>
 <wire x1="34.3154" y1="30.4038" x2="37.2872" y2="33.3756" width="0.254" layer="16"/>
 <wire x1="65.8622" y1="53.4924" x2="66.04" y2="53.34" width="0.254" layer="16"/>
@@
 <contactref element="U$5" pad="4"/>
 <contactref element="U$2" pad="D3"/>
-<wire x1="28.1432" y1="54.4068" x2="28.1432" y2="33.8328" width="0.254" layer="16"/>
-<wire x1="46.8884" y1="73.152" x2="28.1432" y2="54.4068" width="0.254" layer="16"/>
-<wire x1="46.8884" y1="77.9526" x2="46.8884" y2="73.152" width="0.254" layer="16"/>
 <wire x1="47.5742" y1="78.6384" x2="46.8884" y2="77.9526" width="0.254" layer="16"/>
 <wire x1="54.6608" y1="78.6384" x2="47.5742" y2="78.6384" width="0.254" layer="16"/>
@@
 <wire x1="28.1432" y1="33.8328" x2="27.94" y2="33.655" width="0.254" layer="16"/>
 <wire x1="55.8038" y1="77.4954" x2="55.88" y2="77.47" width="0.254" layer="16"/>
+<wire x1="46.8884" y1="77.9526" x2="46.8376" y2="77.9018" width="0.1524" layer="16"/>
+<wire x1="46.8376" y1="77.9018" x2="46.8376" y2="77.00706875" width="0.1524" layer="16"/>
+<wire x1="46.8376" y1="77.00706875" x2="39.525265625" y2="69.694734375" width="0.2032" layer="16"/>
+<wire x1="39.525265625" y1="69.694734375" x2="36.93873125" y2="67.1082" width="0.254" layer="16"/>
+<wire x1="27.94" y1="58.10946875" x2="27.94" y2="33.655" width="0.254" layer="16"/>
+<wire x1="33.343275" y1="67.1082" x2="31.8248" y2="65.589725" width="0.254" layer="16"/>
+<wire x1="31.8248" y1="61.99426875" x2="27.94" y2="58.10946875" width="0.254" layer="16"/>
+<wire x1="36.93873125" y1="67.1082" x2="33.343275" y2="67.1082" width="0.254" layer="16"/>
+<wire x1="31.8248" y1="65.589725" x2="31.8248" y2="61.99426875" width="0.254" layer="16"/>
 </signal>
 </signals>

Commit message: pcb besteld
Other:
- board size 56.8 x 53.3 mm -> 58.1 x 54.6 mm
Changed lines of the file:
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@@
 <board>
 <plain>
-<wire x1="12.7" y1="26.67" x2="69.52" y2="26.67" width="0" layer="20"/>
-<wire x1="69.52" y1="26.67" x2="69.52" y2="80" width="0" layer="20"/>
-<wire x1="69.52" y1="80" x2="12.7" y2="80" width="0" layer="20"/>
-<wire x1="12.7" y1="80" x2="12.7" y2="26.67" width="0" layer="20"/>
+<wire x1="12.7" y1="25.4" x2="70.79" y2="25.4" width="0" layer="20"/>
+<wire x1="70.79" y1="25.4" x2="70.79" y2="80" width="0" layer="20"/>
+<wire x1="70.79" y1="80" x2="12.7" y2="80" width="0" layer="20"/>
+<wire x1="12.7" y1="80" x2="12.7" y2="25.4" width="0" layer="20"/>
 </plain>
 <attributes>
